Commit message: change steering speed limit and speed

File: f1tenth_description/gazebo/ackermann.gazebo.xacro (robot description, xacro)
@@ -15,5 +15,5 @@
             <wheel_base>0.315</wheel_base>
             <wheel_separation>0.2050</wheel_separation>
-            <steer_p_gain>5.0</steer_p_gain>
+            <steer_p_gain>10.0</steer_p_gain>
             <wheel_radius>0.05475</wheel_radius>
             <min_velocity>-3</min_velocity>

File: f1tenth_description/urdf/joints.xacro (robot description, xacro)
@@ -6,6 +6,6 @@
         <parent link="base_link" />
         <axis xyz="0 0 1" />
-        <limit lower="-0.6" upper="+0.6"
-               velocity="1.0" effort="25" />
+        <limit lower="-0.55" upper="+0.55"
+               velocity="3.66" effort="25" />
         <origin xyz="0.1575 0.1025 0.055" rpy="0 0 0"/>
     </joint>
@@ -14,6 +14,6 @@
         <parent link="base_link" />
         <axis xyz="0 0 1" />
-        <limit lower="-0.6" upper="+0.6"
-               velocity="1.0" effort="25" />
+        <limit lower="-0.55" upper="+0.55"
+               velocity="3.66" effort="25" />
         <origin xyz="0.1575 -0.1025 0.055" rpy="0 0 0"/>
     </joint>

Commit message: Corrected wheelbase, wheel separation & steering limit

File: f1tenth_description/gazebo/ackermann.gazebo.xacro (robot description, xacro)
@@ -5,14 +5,18 @@
             filename="gz-sim-ackermann-steering-system"
             name="gz::sim::systems::AckermannSteering">
-            <left_joint>front_left_wheel_joint</left_joint>
+            <!-- <left_joint>front_left_wheel_joint</left_joint> -->
             <left_joint>rear_left_wheel_joint</left_joint>
-            <right_joint>front_right_wheel_joint</right_joint>
+            <!-- <right_joint>front_right_wheel_joint</right_joint> -->
             <right_joint>rear_right_wheel_joint</right_joint>
             <left_steering_joint>front_left_wheel_steering_joint</left_steering_joint>
             <right_steering_joint>front_right_wheel_steering_joint</right_steering_joint>
             <kingpin_width>0.2050</kingpin_width>
-            <steering_limit>0.4667</steering_limit>
-            <wheel_base>0.315</wheel_base>
-            <wheel_separation>0.2050</wheel_separation>
+            <steering_limit>0.4347</steering_limit>
+            <!-- https://gazebosim.org/api/gazebo/6/classignition_1_1gazebo_1_1systems_1_1AckermannSteering.html-->
+            <!-- SPECIAL ATTENTION TO STEERING LIMIT-->
+            <!-- USING TAN, check gz-sim source code, turn radius of ~0.7m -->
+            <wheel_base>0.325</wheel_base>
+            <!-- SHOULD BE MORE WHEEL SEPERATION I.E. TIRE CENTER-->
+            <wheel_separation>0.2450</wheel_separation>
             <steer_p_gain>10.0</steer_p_gain>
             <wheel_radius>0.05475</wheel_radius>

File: f1tenth_description/urdf/const.xacro (robot description, xacro)
@@ -13,5 +13,5 @@
     <xacro:property name="chassis_height" value="0.09" />
     <!-- Joint placement -->
-    <xacro:property name="chassis_to_wheel_x" value="${0.31 /2}" />
+    <xacro:property name="chassis_to_wheel_x" value="${0.325 /2}" />
     <xacro:property name="chassis_to_wheel_y" value="${0.005+ (wheel_width /2) + (chassis_width /2)}" />
     <xacro:property name="chassis_to_wheel_z" value="${wheel_diameter /2}" />

File: f1tenth_description/urdf/joints.xacro (robot description, xacro)
@@ -6,5 +6,5 @@
         <parent link="base_link" />
         <axis xyz="0 0 1" />
-        <limit lower="-0.6" upper="+0.6"
+        <limit lower="-0.7" upper="+0.7"
                velocity="3.66" effort="25" />
         <origin xyz="0.1575 0.1025 0.055" rpy="0 0 0"/>
@@ -14,5 +14,5 @@
         <parent link="base_link" />
         <axis xyz="0 0 1" />
-        <limit lower="-0.6" upper="+0.6"
+        <limit lower="-0.7" upper="+0.7"
                velocity="3.66" effort="25" />
         <origin xyz="0.1575 -0.1025 0.055" rpy="0 0 0"/>
