Commit message: corrected max steering joing angle

File: f1tenth_description/urdf/joints.xacro (robot description, xacro)
@@ -6,5 +6,5 @@
         <parent link="base_link" />
         <axis xyz="0 0 1" />
-        <limit lower="-0.55" upper="+0.55"
+        <limit lower="-0.6" upper="+0.6"
                velocity="3.66" effort="25" />
         <origin xyz="0.1575 0.1025 0.055" rpy="0 0 0"/>
@@ -14,5 +14,5 @@
         <parent link="base_link" />
         <axis xyz="0 0 1" />
-        <limit lower="-0.55" upper="+0.55"
+        <limit lower="-0.6" upper="+0.6"
                velocity="3.66" effort="25" />
         <origin xyz="0.1575 -0.1025 0.055" rpy="0 0 0"/>

Commit message: Added IMU simulation

File: f1tenth_description/urdf/joints.xacro (robot description, xacro)
@@ -58,3 +58,8 @@
         <origin xyz="0.1 0 0.15" rpy="0 0 0"/>
     </joint>
+    <joint name="imu_sensor_joint" type="fixed">
+        <child link="imu_sensor_link"/>
+        <parent link="base_link"/>
+        <origin xyz="0 0 0" rpy="0 0 0"/>
+    </joint>
 </robot>

File: f1tenth_description/urdf/links.xacro (robot description, xacro)
@@ -1,5 +1,6 @@
 <?xml version='1.0'?>
 <robot xmlns:xacro="http://www.ros.org/wiki/xacro">
-    <link name="base_link" />
+    <link name="base_link">
+    </link>
     <!-- Wheels -->
     <xacro:cylinder_link name="front_left_wheel" mesh_file="package://f1tenth_description/meshes/wheel.stl"
@@ -41,3 +42,7 @@
       <origin xyz="0 0 0" rpy="0 0 0"/>
     </xacro:cylinder_link_nomesh>
+    <link name="imu_sensor_link">
+        <gravity>false</gravity>
+        <origin xyz="0 0 0" rpy="0 0 0"/>
+    </link>
 </robot>

File: f1tenth_description/urdf/robot.urdf.xacro (robot description, xacro)
@@ -5,4 +5,5 @@
     <xacro:include filename="$(find f1tenth_description)/urdf/macro.xacro" />
     <xacro:include filename="$(find f1tenth_description)/gazebo/lidar.gazebo.xacro" />
+    <xacro:include filename="$(find f1tenth_description)/gazebo/imu.gazebo.xacro" />
     <!-- links and joints -->
     <xacro:include filename="$(find f1tenth_description)/urdf/links.xacro" />

Commit message: Working aruco marker

File: f1tenth_description/urdf/joints.xacro (robot description, xacro)
@@ -47,4 +47,9 @@
         <origin xyz="-0.1554 0.09 0.2" rpy="0 0 0"/>
     </joint>
+    <joint name="aruco_to_box" type="fixed">
+        <child link="aruco_visual" />
+        <parent link="box_visual" />
+        <origin xyz="-0.016 -0.146 0" rpy="0 ${pi/2} 0"/>
+    </joint>
     <joint name="base_link_to_lower_chassis" type="fixed">
         <child link="lower_chassis" />

File: f1tenth_description/urdf/links.xacro (robot description, xacro)
@@ -37,4 +37,8 @@
         <origin xyz="0 -0.0915 0" rpy="0 0 0"/>
     </xacro:box_link_nomesh >
+    <xacro:box_link name="aruco_visual" mesh_file="package://f1tenth_description/meshes/aruco.stl"
+                    x="0.03" y="0.183" z="0.31 " mass="0.08">
+        <origin xyz="0 0 0" rpy="0 0 0"/>
+    </xacro:box_link>
     <!-- Sensor links -->
     <xacro:cylinder_link_nomesh name="hokuyo_10lx_lidar_link"

File: f1tenth_description/urdf/robot.urdf.xacro (robot description, xacro)
@@ -1,4 +1,5 @@
 <?xml version='1.0'?>
 <robot name="robot" xmlns:xacro="http://www.ros.org/wiki/xacro">
+    <!-- <xacro:include filename="$(find f1tenth_description)/urdf/robot.gazebo.xacro"/> -->
     <!-- Contestants and stuff -->
     <xacro:include filename="$(find f1tenth_description)/urdf/const.xacro" />

Commit message: Should render camera but stl doesn't render

File: f1tenth_description/urdf/joints.xacro (robot description, xacro)
@@ -57,4 +57,9 @@
         <origin xyz="-0.155 0.09 0.055" rpy="0 0 0"/>
     </joint>
+    <joint name="base_link_to_camera" type="fixed">
+        <child link="camera_visual" />
+        <parent link="base_link" />
+        <origin xyz="0.5 0 0" rpy="0 0 0"/>
+    </joint>
     <!-- Sensor Joints -->
     <joint name="hokuyo_10lx_lidar_joint" type="fixed">

File: f1tenth_description/urdf/links.xacro (robot description, xacro)
@@ -41,4 +41,8 @@
         <origin xyz="0 0 0" rpy="0 0 0"/>
     </xacro:box_link>
+    <xacro:box_link name="camera_visual" mesh_file="package://f1tenth_description/meshes/camera.stl"
+                    x="0" y="0" z="0" mass="0.08">
+        <origin xyz="0 0 0" rpy="0 0 0"/>
+    </xacro:box_link>
     <!-- Sensor links -->
     <xacro:cylinder_link_nomesh name="hokuyo_10lx_lidar_link"

Commit message: Camera positioning

File: f1tenth_description/urdf/joints.xacro (robot description, xacro)
@@ -60,5 +60,5 @@
         <child link="camera_visual" />
         <parent link="base_link" />
-        <origin xyz="0.5 0 0" rpy="0 0 0"/>
+        <origin xyz="0.15 0 0.1" rpy="0 0 0"/>
     </joint>
     <!-- Sensor Joints -->

File: f1tenth_description/urdf/links.xacro (robot description, xacro)
@@ -41,5 +41,5 @@
         <origin xyz="0 0 0" rpy="0 0 0"/>
     </xacro:box_link>
-    <xacro:box_link_nomesh name="camera_visual" x="0.05" y="0.2" z="0.3" mass="0.08">
+    <xacro:box_link_nomesh name="camera_visual" x="0.03" y="0.1" z="0.05" mass="0.08">
         <origin xyz="0 0 0" rpy="0 0 0"/>
     </xacro:box_link_nomesh>

Commit message: Camera spawns as LiDAR

File: f1tenth_description/urdf/joints.xacro (robot description, xacro)
@@ -57,9 +57,4 @@
         <origin xyz="-0.155 0.09 0.055" rpy="0 0 0"/>
     </joint>
-    <joint name="base_link_to_camera" type="fixed">
-        <child link="camera_visual" />
-        <parent link="base_link" />
-        <origin xyz="0.15 0 0.1" rpy="0 0 0"/>
-    </joint>
     <!-- Sensor Joints -->
     <joint name="hokuyo_10lx_lidar_joint" type="fixed">
@@ -67,4 +62,9 @@
         <parent link="base_link" />
         <origin xyz="0.1 0 0.15" rpy="0 0 0"/>
+    </joint>
+    <joint name="camera_joint" type="fixed">
+        <child link="camera_link" />
+        <parent link="base_link" />
+        <origin xyz="0.15 0 0.1" rpy="0 0 0"/>
     </joint>
     <joint name="imu_sensor_joint" type="fixed">

File: f1tenth_description/urdf/links.xacro (robot description, xacro)
@@ -41,7 +41,4 @@
         <origin xyz="0 0 0" rpy="0 0 0"/>
     </xacro:box_link>
-    <xacro:box_link_nomesh name="camera_visual" x="0.03" y="0.1" z="0.05" mass="0.08">
-        <origin xyz="0 0 0" rpy="0 0 0"/>
-    </xacro:box_link_nomesh>
     <!-- Sensor links -->
     <xacro:cylinder_link_nomesh name="hokuyo_10lx_lidar_link"
@@ -49,4 +46,7 @@
       <origin xyz="0 0 0" rpy="0 0 0"/>
     </xacro:cylinder_link_nomesh>
+    <xacro:box_link_nomesh name="camera_link" x="0.03" y="0.1" z="0.05" mass="0.08">
+        <origin xyz="0 0 0" rpy="0 0 0"/>
+    </xacro:box_link_nomesh>
     <link name="imu_sensor_link">
         <gravity>false</gravity>

File: f1tenth_description/urdf/robot.urdf.xacro (robot description, xacro)
@@ -6,4 +6,5 @@
     <xacro:include filename="$(find f1tenth_description)/gazebo/lidar.gazebo.xacro" />
     <xacro:include filename="$(find f1tenth_description)/gazebo/imu.gazebo.xacro" />
+    <xacro:include filename="$(find f1tenth_description)/gazebo/camera.gazebo.xacro" />
     <!-- links and joints -->
     <xacro:include filename="$(find f1tenth_description)/urdf/links.xacro" />
