Commit message: camera flag

File: f1tenth_description/urdf/robot.urdf.xacro (robot description, xacro)
@@ -2,4 +2,5 @@
 <robot name="robot" xmlns:xacro="http://www.ros.org/wiki/xacro">
     <xacro:arg name="enable_camera" default="false" />
+    <xacro:property name="enable_camera_flag" value="$(arg enable_camera)" />
     <!-- Contestants and stuff -->
     <xacro:include filename="$(find f1tenth_description)/urdf/const.xacro" />
@@ -7,5 +8,5 @@
     <xacro:include filename="$(find f1tenth_description)/gazebo/lidar.gazebo.xacro" />
     <xacro:include filename="$(find f1tenth_description)/gazebo/imu.gazebo.xacro" />
-    <xacro:if value="${enable_camera == 'true'}">
+    <xacro:if value="${enable_camera_flag == 'true'}">
         <xacro:include filename="$(find f1tenth_description)/gazebo/camera.gazebo.xacro" />
     </xacro:if>

Commit message: launch

File: f1tenth_description/urdf/robot.urdf.xacro (robot description, xacro)
@@ -2,5 +2,4 @@
 <robot name="robot" xmlns:xacro="http://www.ros.org/wiki/xacro">
     <xacro:arg name="enable_camera" default="false" />
-    <xacro:property name="enable_camera_flag" value="$(arg enable_camera)" />
     <!-- Contestants and stuff -->
     <xacro:include filename="$(find f1tenth_description)/urdf/const.xacro" />
@@ -8,5 +7,5 @@
     <xacro:include filename="$(find f1tenth_description)/gazebo/lidar.gazebo.xacro" />
     <xacro:include filename="$(find f1tenth_description)/gazebo/imu.gazebo.xacro" />
-    <xacro:if value="${enable_camera_flag == 'true'}">
+    <xacro:if value="$(arg enable_camera)">
         <xacro:include filename="$(find f1tenth_description)/gazebo/camera.gazebo.xacro" />
     </xacro:if>
